File: cheap_boi.kicad_pcb (KiCad board)
At the start: 2 copper layers, 287.3 x 76.2 mm, 136 parts, among them SW1 SW_Push, U1 ATmega32U4-AU, Y1 16MHz

Commit message: added evenly distributed groundfill
Routing:
- added copper zone on B.Cu, net GND
- added copper zone on F.Cu, net GND

Commit message: revised traces that where 90deg and smaller
Routing:
- net +5V: track 660.1 -> 661.8 mm
- net ROW0: track 292.5 -> 293.5 mm

Commit message: add Gerbers + gerber zip
Parts:
- F1: value Polyfuse_Small -> 500mA
Changed lines of the file:
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@@
       (effects (font (size 1 1) (thickness 0.15)) (justify mirror))
     )
-    (fp_text value Polyfuse_Small (at 0 -1.82) (layer B.Fab)
+    (fp_text value 500mA (at 0 -1.82) (layer B.Fab)
       (effects (font (size 1 1) (thickness 0.15)) (justify mirror))
     )
@@
     (connect_pads (clearance 0.508))
     (min_thickness 0.254)
-    (fill (arc_segments 32) (thermal_gap 0.508) (thermal_bridge_width 0.508))
+    (fill yes (arc_segments 32) (thermal_gap 0.508) (thermal_bridge_width 0.508))
     (polygon
       (pts
@@
     (connect_pads (clearance 0.508))
     (min_thickness 0.254)
-    (fill (arc_segments 32) (thermal_gap 0.508) (thermal_bridge_width 0.508))
+    (fill yes (arc_segments 32) (thermal_gap 0.508) (thermal_bridge_width 0.508))
     (polygon
       (pts

Commit message: imagine a good commit message, don't have time
Parts:
- moved REF** 0.28 mm to (235.7, 71.4)
- moved REF** 0.26 mm to (81.8, 71.4)
- moved REF** 0.07 mm to (331.0, 71.4)
- moved REF** 0.07 mm to (140.5, 71.4)
Changed lines of the file:
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@@
     (visible_elements FFFFFF7F)
     (pcbplotparams
-      (layerselection 0x010fc_ffffffff)
-      (usegerberextensions false)
+      (layerselection 0x010f0_ffffffff)
+      (usegerberextensions true)
       (usegerberattributes true)
       (usegerberadvancedattributes true)
-      (creategerberjobfile true)
+      (creategerberjobfile false)
       (excludeedgelayer true)
       (linewidth 0.100000)
@@
       (plotinvisibletext false)
       (padsonsilk false)
-      (subtractmaskfromsilk false)
+      (subtractmaskfromsilk true)
       (outputformat 1)
       (mirror false)
-      (drillshape 1)
+      (drillshape 0)
       (scaleselection 1)
-      (outputdirectory ""))
+      (outputdirectory "gerber_files"))
   )
   (net 0 "")
@@
   )
   (module MountingHole:MountingHole_5.3mm_M5 (layer F.Cu)
-    (at 331 71.5)
+    (at 330.9729 71.433)
     (descr "Mounting Hole 5.3mm, no annular, M5")
     (tags "mounting hole 5.3mm no annular m5")
@@
   )
   (module MountingHole:MountingHole_5.3mm_M5 (layer F.Cu)
-    (at 236 71.5)
+    (at 235.7289 71.433)
     (descr "Mounting Hole 5.3mm, no annular, M5")
     (tags "mounting hole 5.3mm no annular m5")
@@
   )
   (module MountingHole:MountingHole_5.3mm_M5 (layer F.Cu)
-    (at 140.5 71.5)
+    (at 140.5 71.433)
     (descr "Mounting Hole 5.3mm, no annular, M5")
     (tags "mounting hole 5.3mm no annular m5")
@@
   )
   (module MountingHole:MountingHole_5.3mm_M5 (layer F.Cu)
-    (at 82 71.5)
+    (at 81.7511 71.433)
     (descr "Mounting Hole 5.3mm, no annular, M5")
     (tags "mounting hole 5.3mm no annular m5")
@@
     (connect_pads (clearance 0.508))
     (min_thickness 0.254)
-    (fill yes (arc_segments 32) (thermal_gap 0.508) (thermal_bridge_width 0.508))
+    (fill (arc_segments 32) (thermal_gap 0.508) (thermal_bridge_width 0.508))
     (polygon
       (pts
@@
     (connect_pads (clearance 0.508))
     (min_thickness 0.254)
-    (fill yes (arc_segments 32) (thermal_gap 0.508) (thermal_bridge_width 0.508))
+    (fill (arc_segments 32) (thermal_gap 0.508) (thermal_bridge_width 0.508))
     (polygon
       (pts

Commit message: added new gerbers
Connections:
- USB1 pad 6: Net-(USB1-Pad6) -> GND
Routing:
- net GND: track 689.5 -> 711.9 mm
