File: cheap_boi.kicad_pcb (KiCad board)
At the start: 2 copper layers, 287.3 x 76.2 mm, 136 parts, among them SW1 SW_Push, U1 ATmega32U4-AU, Y1 16MHz

Commit message: we are now on rev 1.1, pcbs soon to be tested
Parts:
- added G***: LOGO, lorax_silk:the_lorax_tree, B.Cu at (165.9, 74.9)
- added G***: LOGO, lorax_silk:the_lorax_mirror, B.Cu at (301.2, 71.4)
- added MX40: MX-NoLED, MX_Alps_Hybrid_2:MX-2U-ReversedStabilizers-NoLED, F.Cu at (235.7, 100.1)
-  : renamed from REF** (x4)
- Y1: footprint Crystal:Crystal_SMD_3225-4Pin_3.2x2.5mm -> Crystal:Crystal_SMD_3225-4Pin_3.2x2.5mm_HandSoldering
- moved D28 4.07 mm to (239.0, 103.9)
- moved C4 1.66 mm to (96.8, 74.6)
- moved Y1 1.58 mm to (101.4, 74.8)
- moved C3 1.53 mm to (106.2, 74.6)
Routing:
- net ROW3: track 315.9 -> 376.6 mm
- net Net-(D28-Pad2): track 9.40 -> 24.1 mm
- net GND: track 711.9 -> 724.4 mm, vias 16 -> 21
- net COL6: track 198.1 -> 209.0 mm
- net COL7: track 238.6 -> 242.8 mm
- net COL11: track 347.7 -> 350.3 mm
- net COL12: track 367.9 -> 370.4 mm
- net COL10: track 322.7 -> 325.1 mm
- net ROW1: track 300.1 -> 302.4 mm
- net COL8: track 261.6 -> 263.8 mm
- net +5V: track 661.8 -> 659.7 mm
- net COL9: track 300.0 -> 302.1 mm
- net Net-(C4-Pad1): track 7.61 -> 9.59 mm
- net Net-(C3-Pad1): track 16.8 -> 15.7 mm
- net VCC: track 72.3 -> 73.3 mm
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Other:
- board text added: "This is the cheap_boi rev 1.1"
- board text added: "Unless someone like you cares a whole awful lot, nothing is going to get better. It's not."
- board text removed: "cheap_boi Rev 1 made by MangoIV, thx to the 40% Discord server for excessive help"
